Commit message: Update Project 2 so the robot is round like a roomba.

File: Project2/my_robot/urdf/my_robot_original.xacro (robot description, xacro)
@@ -13,6 +13,5 @@
         <color rgba="0.75 0.75 0.75 1" />
     </material> -->
-    <!-- Colors from the course -->
-    <!-- <gazebo reference="chassis">
+    <gazebo reference="chassis">
         <material>Gazebo/Blue</material>
     </gazebo>
@@ -25,16 +24,4 @@
     <gazebo reference="left_wheel">
         <material>Gazebo/Green</material>
-    </gazebo> -->
-    <gazebo reference="chassis">
-        <material>Gazebo/Orange</material>
-    </gazebo>
-    <gazebo reference="right_wheel">
-        <material>Gazebo/Turquoise</material>
-    </gazebo>
-    <gazebo reference="left_wheel">
-        <material>Gazebo/Indigo</material>
-    </gazebo>
-    <gazebo reference="camera">
-        <material>Gazebo/Red</material>
     </gazebo>
     <xacro:include filename="$(find my_robot)/urdf/my_robot.gazebo" />
@@ -59,6 +46,5 @@
             <origin xyz="0 0 0" rpy=" 0 0 0"/>
             <geometry>
-                <!-- <box size=".4 .2 .1"/> -->
-                <cylinder length="0.1" radius="0.2" />
+                <box size=".4 .2 .1"/>
             </geometry>
         </collision>
@@ -66,6 +52,5 @@
             <origin xyz="0 0 0" rpy=" 0 0 0"/>
             <geometry>
-                <!-- <box size=".4 .2 .1"/> -->
-                <cylinder length="0.1" radius="0.2" />
+                <box size=".4 .2 .1"/>
             </geometry>
             <!-- <material name="blue" /> -->
@@ -145,5 +130,5 @@
     </link>
     <joint type="continuous" name="left_wheel_hinge">
-        <origin xyz="0 0.23 0" rpy="0 0 0"/>
+        <origin xyz="0 0.15 0" rpy="0 0 0"/>
         <child link="left_wheel"/>
         <parent link="chassis"/>
@@ -153,5 +138,5 @@
     </joint>
     <joint type="continuous" name="right_wheel_hinge">
-        <origin xyz="0 -0.23 0" rpy="0 0 0"/>
+        <origin xyz="0 -0.15 0" rpy="0 0 0"/>
         <child link="right_wheel"/>
         <parent link="chassis"/>

File: catkin_workspace/src/my_robot/urdf/my_robot.xacro (robot description, xacro)
@@ -13,5 +13,6 @@
         <color rgba="0.75 0.75 0.75 1" />
     </material> -->
-    <gazebo reference="chassis">
+    <!-- Colors from the course -->
+    <!-- <gazebo reference="chassis">
         <material>Gazebo/Blue</material>
     </gazebo>
@@ -24,4 +25,16 @@
     <gazebo reference="left_wheel">
         <material>Gazebo/Green</material>
+    </gazebo> -->
+    <gazebo reference="chassis">
+        <material>Gazebo/Orange</material>
+    </gazebo>
+    <gazebo reference="right_wheel">
+        <material>Gazebo/Turquoise</material>
+    </gazebo>
+    <gazebo reference="left_wheel">
+        <material>Gazebo/Indigo</material>
+    </gazebo>
+    <gazebo reference="camera">
+        <material>Gazebo/Red</material>
     </gazebo>
     <xacro:include filename="$(find my_robot)/urdf/my_robot.gazebo" />
@@ -46,5 +59,6 @@
             <origin xyz="0 0 0" rpy=" 0 0 0"/>
             <geometry>
-                <box size=".4 .2 .1"/>
+                <!-- <box size=".4 .2 .1"/> -->
+                <cylinder length="0.1" radius="0.2" />
             </geometry>
         </collision>
@@ -52,5 +66,6 @@
             <origin xyz="0 0 0" rpy=" 0 0 0"/>
             <geometry>
-                <box size=".4 .2 .1"/>
+                <!-- <box size=".4 .2 .1"/> -->
+                <cylinder length="0.1" radius="0.2" />
             </geometry>
             <!-- <material name="blue" /> -->
@@ -130,5 +145,5 @@
     </link>
     <joint type="continuous" name="left_wheel_hinge">
-        <origin xyz="0 0.15 0" rpy="0 0 0"/>
+        <origin xyz="0 0.23 0" rpy="0 0 0"/>
         <child link="left_wheel"/>
         <parent link="chassis"/>
@@ -138,5 +153,5 @@
     </joint>
     <joint type="continuous" name="right_wheel_hinge">
-        <origin xyz="0 -0.15 0" rpy="0 0 0"/>
+        <origin xyz="0 -0.23 0" rpy="0 0 0"/>
         <child link="right_wheel"/>
         <parent link="chassis"/>
